File: Documentation/1-TurretGuts/PCB/wrangler/wrangler.kicad_sch (KiCad schematic)
At the start: 82 parts, among them J1 USB_C_Receptacle, J2 SMA-RP, J3 Trigger Conn, J4 Joystick Conn, J5 LED, J6 BatteryLED, J7 2PolSwitch, J8 18650 BATTERY, J9 Spare Conn, Q1 FS8205A, Q2 AO3401A, U2 TP4056-42-ESOP8, U3 ATmega32U4-A, U4 nRF24L01P, U5 RFX2401C, U6 AMS1117, U8 DW01A, U9 MT3608, Y2 16 MHz, Y3 16MHz

Commit message: wrangler pass 1
Parts:
- removed J3: Trigger Conn, symbol Connector:Conn_01x02_Pin
- removed J4: Joystick Conn, symbol Connector:Conn_01x05_Pin
- removed J5: LED, symbol Connector:Conn_01x02_Pin
- removed J6: BatteryLED, symbol Connector:Conn_01x02_Pin
- removed J7: 2PolSwitch, symbol Connector:Conn_01x03_Pin
- removed J8: 18650 BATTERY, symbol Connector:Conn_01x02_Pin
- removed J9: Spare Conn, symbol Connector:Conn_01x02_Pin
- removed Q1: FS8205A, FS8205A:SOP65P640X120-8N, symbol FS8205A:FS8205A
- removed Y2: 16 MHz, symbol Device:Crystal
- removed Y3: 16MHz, symbol Device:Crystal
- added J-18650, J-BattLED1, J-LED1, J-Spare1, J-Trigger1: 35317-0221, MiniFitJR2x1:353170221, symbol 35317-0221:35317-0221
- added J-Joystick1: 35317-0620, MiniFitJR3x2:RHDR6W107P420_2X3_1380X960X1310P, symbol 35317-0620:35317-0620
- added J-PowerSwitch1: 35317-0420, MiniFitJR2x2:SHDR4W107P420_2X2_960X960X1280P, symbol 35317-0420:35317-0420
- added Q3: FS8205A, Package_TO_SOT_SMD:SOT-23-6, symbol FS8205A:FS8205A
- added Y1, Y2: 16MHz, Crystal:Crystal_SMD_3225-4Pin_3.2x2.5mm, symbol Device:Crystal_GND24
- C1, C10, C11, C12, C13, C14, C15, C16, C17, C18, C19, C20, C21, C22, C23, C24, C25, C26, C27, C28, C29, C30, C31, C32, C4, C5, C6, C7, C8, C9, L1, L2, L3, L4, L6: footprint (none) -> Capacitor_SMD:C_0201_0603Metric
- D10, D11, D12, D9: footprint (none) -> LED_SMD:LED_0805_2012Metric
- J1: footprint (none) -> Connector_USB:USB_C_Receptacle_HRO_TYPE-C-31-M-12
- J2: footprint (none) -> Connector_Coaxial:SMA_Amphenol_132289_EdgeMount
- L5: footprint (none) -> Inductor_SMD:L_1206_3216Metric
- R1, R10, R11, R12, R13, R14, R15, R16, R17, R18, R19, R2, R3, R5, R6, R7, R8, R9: footprint (none) -> Capacitor_SMD:C_0805_2012Metric
Connections:
- net +5.3V: now also J-PowerSwitch1.4
- net +5V: now also J-BattLED1.2, J-LED1.2
- net GND: now also J-BattLED1.1, J-Joystick1.6, J-LED1.1, J-Spare1.1, J-Trigger1.1, Q3.3 (S2), Y1.2, Y1.4, Y2.2, Y2.4
- net GPIO1: now also J-Joystick1.1
- net GPIO2: now also J-Joystick1.2
- net GPIO3: now also J-Joystick1.3
- net GPIO4: now also J-Joystick1.4
- net GPIO5: now also J-Trigger1.2
- net GPIO6: now also J-Spare1.2
- net +V_Batt: now reaches Q2.3 (D), R14.2, U2.5 (BAT)
- net +V_Batt: now also J-18650.2
- net at C11.1, U4.9 (XC2): now also Y1.1
- net at C30.1, U3.16 (XTAL2): now also Y2.3
- net at C12.1, U4.10 (XC1): now also Y1.3
- net at U8.1 (OD): now also Q3.6 (G1)
- net at U8.3 (OC): now also Q3.4 (G2)
- net at C31.1, U3.17 (XTAL1): now also Y2.1
- net HighFlag renamed HighSwitch
- net HighSwitch: now also J-PowerSwitch1.1
- net LowFlag renamed LowSwitch
- net LowSwitch: now also J-PowerSwitch1.2
- new net -V_Batt: J-18650.1, Q3.1 (S1)
- no-connect marks 11 -> 27
Other:
- moved on the sheet: C10, C11, C12, C13, C14, C15, C16, C17, C18, C19, C20, C22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
